File: SmartWasteBin/SmartWasteBin_PCB/SmartWasteBin.sch (KiCad schematic (older format))
At the start: 10 parts, among them P1 CONN_01X04, P10 CONN_01X02, P2 CONN_01X03, P3 CONN_01X03, P4 CONN_01X16, P5 CONN_01X12, P6 CONN_01X07, P7 CONN_01X03, P8 CONN_01X03, P9 CONN_01X04

Commit message: Update PCB
Parts:
- P1, P9: footprint (none) -> CONN:CONN_01x04
- P10: footprint (none) -> CONN:CONN_01x02
- P2, P3, P7, P8: footprint (none) -> CONN:CONN_01x03
- P4: footprint (none) -> CONN:CONN_01x16
- P5: footprint (none) -> CONN:CONN_01x12
- P6: footprint (none) -> CONN:CONN_01x07
Connections:
- net at P4.11 (P11): now also P9.2 (P2); no longer P9.3 (P3)
- net at P4.12 (P12): now also P9.3 (P3); no longer P9.2 (P2)
- net at P4.16 (P16): now also P5.4 (P4); no longer P5.3 (P3)
- net at P7.3 (P3): now also P5.3 (P3); no longer P5.4 (P4)
Changed lines of the file:
@@
 LIBS:contrib
 LIBS:valves
+LIBS:SmartWasteBin-cache
 EELAYER 25 0
 EELAYER END
@@
 F 0 "P4" H 5500 6200 50  0000 C CNN
 F 1 "CONN_01X16" V 5600 5350 50  0000 C CNN
-F 2 "" H 5500 5350 50  0000 C CNN
+F 2 "CONN:CONN_01x16" H 5500 5350 50  0001 C CNN
 F 3 "" H 5500 5350 50  0000 C CNN
 	1    5500 5350
@@
 F 0 "P5" H 5550 4100 50  0000 C CNN
 F 1 "CONN_01X12" V 5650 3450 50  0000 C CNN
-F 2 "" H 5550 3450 50  0000 C CNN
+F 2 "CONN:CONN_01x12" H 5550 3450 50  0001 C CNN
 F 3 "" H 5550 3450 50  0000 C CNN
 	1    5550 3450
@@
 F 0 "P6" H 6100 2150 50  0000 C CNN
 F 1 "CONN_01X07" V 6200 1750 50  0000 C CNN
-F 2 "" H 6100 1750 50  0000 C CNN
+F 2 "CONN:CONN_01x07" H 6100 1750 50  0001 C CNN
 F 3 "" H 6100 1750 50  0000 C CNN
 	1    6100 1750
@@
 F 0 "P8" H 7700 2600 50  0000 C CNN
 F 1 "CONN_01X03" V 7800 2400 50  0000 C CNN
-F 2 "" H 7700 2400 50  0000 C CNN
+F 2 "CONN:CONN_01x03" H 7700 2400 50  0001 C CNN
 F 3 "" H 7700 2400 50  0000 C CNN
 	1    7700 2400
@@
 F 0 "P2" H 3000 2500 50  0000 C CNN
 F 1 "CONN_01X03" V 3100 2300 50  0000 C CNN
-F 2 "" H 3000 2300 50  0000 C CNN
+F 2 "CONN:CONN_01x03" H 3000 2300 50  0001 C CNN
 F 3 "" H 3000 2300 50  0000 C CNN
 	1    3000 2300
@@
 F 0 "P1" H 2750 4600 50  0000 C CNN
 F 1 "CONN_01X04" V 2850 4350 50  0000 C CNN
-F 2 "" H 2750 4350 50  0000 C CNN
+F 2 "CONN:CONN_01x04" H 2750 4350 50  0001 C CNN
 F 3 "" H 2750 4350 50  0000 C CNN
 	1    2750 4350
@@
 F 0 "P9" H 8550 4800 50  0000 C CNN
 F 1 "CONN_01X04" V 8650 4550 50  0000 C CNN
-F 2 "" H 8550 4550 50  0000 C CNN
+F 2 "CONN:CONN_01x04" H 8550 4550 50  0001 C CNN
 F 3 "" H 8550 4550 50  0000 C CNN
 	1    8550 4550
@@
 F 0 "P3" H 3750 2700 50  0000 C CNN
 F 1 "CONN_01X03" V 3850 2500 50  0000 C CNN
-F 2 "" H 3750 2500 50  0000 C CNN
+F 2 "CONN:CONN_01x03" H 3750 2500 50  0001 C CNN
 F 3 "" H 3750 2500 50  0000 C CNN
 	1    3750 2500
@@
 F 0 "P10" H 8650 3500 50  0000 C CNN
 F 1 "CONN_01X02" V 8750 3350 50  0000 C CNN
-F 2 "" H 8650 3350 50  0000 C CNN
+F 2 "CONN:CONN_01x02" H 8650 3350 50  0001 C CNN
 F 3 "" H 8650 3350 50  0000 C CNN
 	1    8650 3350
@@
 F 0 "P7" H 6800 4600 50  0000 C CNN
 F 1 "CONN_01X03" V 6900 4400 50  0000 C CNN
-F 2 "" H 6800 4400 50  0000 C CNN
+F 2 "CONN:CONN_01x03" H 6800 4400 50  0001 C CNN
 F 3 "" H 6800 4400 50  0000 C CNN
 	1    6800 4400
@@
 	6400 5650 6400 3100
 Wire Wire Line
-	6400 3100 5900 3100
-Wire Wire Line
-	5900 3100 5900 3250
-Wire Wire Line
 	7000 4300 7100 4300
 Wire Wire Line
 	7100 4300 7100 3000
-Wire Wire Line
-	7100 3000 5800 3000
-Wire Wire Line
-	5800 3000 5800 3250
 Wire Wire Line
 	5800 1950 5800 2550
@@
 	8350 4500 7900 4500
 Wire Wire Line
-	7900 4500 7900 6350
-Wire Wire Line
-	7900 6350 5850 6350
-Wire Wire Line
-	5850 6350 5850 5550
-Wire Wire Line
-	8350 4600 8150 4600
-Wire Wire Line
-	8150 4600 8150 6450
-Wire Wire Line
-	8150 6450 5750 6450
-Wire Wire Line
-	5750 6450 5750 5550
+	8050 4600 8350 4600
 Wire Wire Line
 	4850 5800 4850 5550
@@
 	7700 4700 7700 3700
 Connection ~ 7700 3700
+Wire Wire Line
+	7100 3000 5900 3000
+Wire Wire Line
+	5900 3000 5900 3250
+Wire Wire Line
+	6400 3100 5800 3100
+Wire Wire Line
+	5800 3100 5800 3250
+Wire Wire Line
+	7900 4500 7900 6200
+Wire Wire Line
+	7900 6200 5750 6200
+Wire Wire Line
+	5750 6200 5750 5550
+Wire Wire Line
+	8050 4600 8050 6350
+Wire Wire Line
+	5850 6350 8050 6350
+Wire Wire Line
+	5850 5550 5850 6350
 $EndSCHEMATC
